Commit message: feat: Sensor upgrade to depth camera

File: my_robot/urdf/my_robot.xacro (robot description, xacro)
@@ -146,4 +146,11 @@
     <child link="camera" />
   </joint>
+  <joint name="camera_optical_joint" type="fixed">
+    <origin xyz="0 0 0" rpy="-1.5707 0 -1.5707"/>
+    <parent link="camera"/>
+    <child link="camera_link_optical"/>
+  </joint>
+  <link name="camera_link_optical">
+  </link>
   <link name='hokuyo'>
     <inertial>
